File: surse KiCad/Proiect_SDTR2023/Proiect_SDTR2023.kicad_sch (KiCad schematic)
At the start: 3 parts, among them U3 NUCLEO-F401RE

Commit message: few functional fixes.
Parts:
- removed U1: ~, symbol Proj_SDTR_SYMBOL:HC-05
- removed unit 6 of U3
- removed unit 5 of U3
- removed unit 4 of U3
- U2: value ~ -> HC-SR04
Connections:
- net at U3.CN10_15 (PA7): now also U2.3 (ECHO)
- net at U2.1 (VCC): now also U3.CN6_5 (+5V)
- net at U2.2 (TRIG): now also U3.CN7_32 (PA4)
- net at U2.4 (GND): now also U3.CN6_6 (GND), U3.CN6_7 (GND)
Other:
- moved on the sheet: U2, U3A, U3B, U3C
